Commit message: Restructure: move package files into autonomus_navigation/ subfolder for standard ROS2 layout

File: autonomus_navigation/description/robot.urdf.xacro (robot description, xacro)
@@ -2,4 +2,5 @@
 <robot xmlns:xacro="http://www.ros.org/wiki/xacro"  name="robot">
 <xacro:include filename="robot_core.xacro" />
+<xacro:include filename="gazebo_control.xacro" />
     <!-- Example link -->
 </robot>

File: autonomus_navigation/description/robot_core.xacro (robot description, xacro)
@@ -110,3 +110,8 @@
     </xacro:inertial_sphere>
     </link>
+    <gazebo reference="caster_wheel_link">
+        <material>Gazebo/Black</material>
+        <mu1>0.001</mu1>
+        <mu2>0.001</mu2>
+    </gazebo>
 </robot>
